File: new-pcb/tud-microled-v2.kicad_pcb (KiCad board)
At the start: 2 copper layers, 100 x 100 mm, 187 parts

Commit message: Refactor code structure for improved readability and maintainability
Parts:
- moved FID4 7.07 mm to (91.0, 91.0)
- moved PP_GND4 5.83 mm to (88.0, 89.5)
- moved PP_GND2 5.22 mm to (88.0, 16.0)
- moved D1 5.15 mm to (12.5, 78.0)
- moved D2 5.15 mm to (22.5, 78.0)
- moved D3 5.15 mm to (32.5, 78.0)
- moved D4 5.15 mm to (42.5, 78.0)
- moved D5 5.15 mm to (52.5, 78.0)
- moved D6 5.15 mm to (62.5, 78.0)
- moved D7 5.15 mm to (72.5, 78.0)
- moved D8 5.15 mm to (82.5, 78.0)
- moved PP_D1_A 5.15 mm to (9.50, 81.0)
- moved PP_D1_KB 5.15 mm to (13.5, 81.0)
- moved PP_D1_KG 5.15 mm to (11.5, 81.0)
- moved PP_D1_KR 5.15 mm to (15.5, 81.0)
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Connections:
- H_N_1 pad 1: (no net) -> DCL6_IN
- H_N_10 pad 1: (no net) -> DCL6_OUT
- H_N_22 pad 1: (no net) -> DCL12_IN
- H_N_30 pad 1: (no net) -> DCL12_OUT
Routing:
- net DCL12_IN: track 5.90 -> 75.1 mm
- net DCL6_OUT: track 5.90 -> 67.8 mm
- net DCL6_IN: track 5.90 -> 67.6 mm
- net DCL12_OUT: track 5.90 -> 66.7 mm
- net LED_VCC: track 144.1 -> 148.1 mm
- net LED6_KR: track 9.50 -> 10.0 mm
- net LED6_KG: track 6.38 -> 6.88 mm
- net LED6_KB: track 6.86 -> 7.36 mm
- net LED3_KG: track 6.86 -> 7.36 mm
- net LED8_KR: track 9.82 -> 10.3 mm
- net LED8_KG: track 6.64 -> 7.14 mm
- net LED8_KB: track 7.18 -> 7.68 mm
- net LED7_KR: track 9.66 -> 10.2 mm
- net LED7_KG: track 6.48 -> 6.98 mm
- net LED7_KB: track 7.02 -> 7.52 mm
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Other:
- board size 100 x 100 mm -> 95 x 95 mm
- board text added: "95 x 95 mm - 2-layer FR-4 - ENIG (all pads gold)"
- board text added: "TIER-2 NORTH - pins 1,10,22,30 -> LED chains; others jumperable"
- board text added: "TIER-2 SOUTH - pre-wired to LEDs D1..D8 - 32 pins @ 2.54 mm"
- board text added: "W=0.1"
- board text added: "W=0.25"
- board text added: "W=0.5"
- board text added: "W=1.0"
- board text removed: "0"
- board text removed: "100 x 100 mm - 2-layer FR-4 - ENIG (all pads gold)"
- board text removed: "40"
- board text removed: "50"
- board text removed: "60"
- board text removed: "70"
- board text removed: "80"
- board text removed: "TIER-2 NORTH - user-jumperable - 30 pins @ 2.54 mm"
- board text removed: "TIER-2 SOUTH - pre-wired to LEDs D1..D7 - 30 pins @ 2.54 mm"
- board text removed: "VDP W = 0.1 mm"
- board text removed: "VDP W = 0.25 mm"
- board text removed: "VDP W = 0.5 mm"
- board text removed: "VDP W = 1.0 mm"
- board text removed: "WL-SFCC 0404 RGB LEDs"

Commit message: Refactor code structure for improved readability and maintainability
Parts:
- removed PP_GND3: PP_GND3, Probe_1.27mm
- removed PP_GND4: PP_GND4, Probe_1.27mm
- added H_N_31: H_N_31, Header_2.54mm, F.Cu at (83.3, 13.5)
- added H_N_32: H_N_32, Header_2.54mm, F.Cu at (85.9, 13.5)
- moved TC1 4.00 mm to (2.50, 50.5)
- moved TC2 4.00 mm to (2.50, 64.5)
- moved H_N_16 3.54 mm to (45.2, 13.5)
- moved H_N_22 3.54 mm to (60.5, 13.5)
- moved H_N_24 3.54 mm to (65.5, 13.5)
- moved H_N_26 3.54 mm to (70.6, 13.5)
- moved H_N_28 3.54 mm to (75.7, 13.5)
- moved H_N_29 3.54 mm to (78.2, 13.5)
- moved H_N_10 3.54 mm to (30.0, 13.5)
- moved H_N_6 3.54 mm to (19.8, 13.5)
- moved H_N_2 3.54 mm to (9.67, 13.5)
- moved H_N_1 3.54 mm to (7.13, 13.5)
- moved H_N_11 3.54 mm to (32.5, 13.5)
- moved H_N_12 3.54 mm to (35.1, 13.5)
- moved H_N_13 3.54 mm to (37.6, 13.5)
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Connections:
- H_N_1 pad 1: DCL6_IN -> (no net)
- H_N_19 pad 1: (no net) -> DCL12_IN
- H_N_22 pad 1: DCL12_IN -> (no net)
- H_N_3 pad 1: (no net) -> DCL6_IN
- H_N_30 pad 1: DCL12_OUT -> (no net)
Routing:
- net DCL12_IN: track 75.1 -> 65.9 mm
- net DCL6_OUT: track 67.8 -> 65.6 mm
- net DCL6_IN: track 67.6 -> 66.0 mm
- net DCL12_OUT: track 66.7 -> 65.2 mm
- net GND: vias 8 -> 6
Other:
- board size 95 x 95 mm -> 93 x 93 mm
- board text added: "0"
- board text added: "40"
- board text added: "50"
- board text added: "60"
- board text added: "70"
- board text added: "93 x 93 mm - 2-layer FR-4 - ENIG (all pads gold)"
- board text added: "NORTH 32-pin - O = pre-wired LED chain (others jumperable)"
- board text removed: "95 x 95 mm - 2-layer FR-4 - ENIG (all pads gold)"
- board text removed: "TH1"
- board text removed: "TH2"
- board text removed: "TH3"
- board text removed: "TH4"
- board text removed: "TIER-2 NORTH - pins 1,10,22,30 -> LED chains; others jumperable"
- board text removed: "W=0.1"
- board text removed: "W=0.25"
- board text removed: "W=0.5"
- board text removed: "W=1.0"

Commit message: Refactor code structure for improved readability and maintainability
Parts:
- moved PP_DCL12_IN 1.50 mm to (53.9, 72.0)
- moved PP_DCL12_OUT 1.50 mm to (86.2, 72.0)
- moved PP_DCL6_IN 1.50 mm to (13.3, 72.0)
- moved PP_DCL6_OUT 1.50 mm to (30.6, 72.0)
- moved PP_NTC1 0.30 mm to (17.5, 76.8)
- moved PP_NTC2 0.30 mm to (37.5, 76.8)
- moved PP_NTC3 0.30 mm to (57.5, 76.8)
- moved PP_NTC4 0.30 mm to (77.5, 76.8)
- moved TH1 0.30 mm to (20.0, 76.8)
- moved TH2 0.30 mm to (40.0, 76.8)
- moved TH3 0.30 mm to (60.0, 76.8)
- moved TH4 0.30 mm to (80.0, 76.8)
Routing:
- net DCL6_OUT: track 65.6 -> 63.6 mm
- net DCL6_IN: track 66.0 -> 64.0 mm
- net DCL12_OUT: track 65.2 -> 63.2 mm
- net DCL12_IN: track 65.9 -> 63.9 mm
Other:
- board text added: "TH1"
- board text added: "TH2"
- board text added: "TH3"
- board text added: "TH4"

Commit message: Refactor code structure for improved readability and maintainability
Other:
- board text added: "NORTH 3,10,19,32 = pre-wired chain (others jumperable)"
- board text removed: "NORTH row: user-jumperable"
