File: new-pcb/tud-microled-v2.kicad_pcb (KiCad board)
At the start: 2 copper layers, 93 x 93 mm, 187 parts

Commit message: Refactor code structure for improved readability and maintainability
Parts:
- added PP_EIS_LOAD_A: PP_EIS_LOAD_A, Probe_1.27mm, F.Cu at (71.0, 32.5)
- added PP_EIS_LOAD_B: PP_EIS_LOAD_B, Probe_1.27mm, F.Cu at (73.0, 32.5)
- added PP_EIS_OPEN_A: PP_EIS_OPEN_A, Probe_1.27mm, F.Cu at (51.0, 32.5)
- added PP_EIS_OPEN_B: PP_EIS_OPEN_B, Probe_1.27mm, F.Cu at (54.0, 32.5)
- added PP_EIS_SHORT_A: PP_EIS_SHORT_A, Probe_1.27mm, F.Cu at (61.0, 32.5)
- added PP_EIS_SHORT_B: PP_EIS_SHORT_B, Probe_1.27mm, F.Cu at (64.0, 32.5)
Routing:
- net EIS_SHORT: track 0.00 -> 3.00 mm
Other:
- board text added: "100R LOAD"
- board text added: "C1,4: R=50um C2,5: R=100um C3,6: R=200um"
- board text added: "DoE LEGEND"
- board text added: "EIS CAL"
- board text added: "OPEN"
- board text added: "PCB v4.0 / ECTM + ITEC / 2026"
- board text added: "R1-2: plain R3-4: +4 mini R5-6: rounded+mini"
- board text added: "SHORT"
- board text added: "calibrate LCR meter before EIS Nyquist sweep"
- board text removed: "C1, C4 : R = 50 um"
- board text removed: "C2, C5 : R = 100 um"
- board text removed: "C3, C6 : R = 200 um"
- board text removed: "LEGEND"
- board text removed: "PCB v2.0 / ECTM + ITEC / 2026"
- board text removed: "R1, R2 : plain"
- board text removed: "R3, R4 : + 4 minis"
- board text removed: "R5, R6 : rounded + minis"

Commit message: Refactor code structure for improved readability and maintainability
Connections:
- H_N_13 pad 1: (no net) -> NTC2
- H_N_21 pad 1: (no net) -> NTC3
- H_N_29 pad 1: (no net) -> NTC4
- H_N_5 pad 1: (no net) -> NTC1
Routing:
- net NTC4: track 2.00 -> 66.0 mm, vias 0 -> 1
- net NTC3: track 2.00 -> 65.7 mm, vias 0 -> 1
- net NTC1: track 2.00 -> 65.5 mm, vias 0 -> 1
- net NTC2: track 2.00 -> 65.4 mm, vias 0 -> 1
Other:
- board text added: "NORTH 32-pin - O = pre-wired (4 LED chain + 4 NTC), others jumperable"
- board text removed: "NORTH 32-pin - O = pre-wired LED chain (others jumperable)"

Commit message: Refactor code structure for improved readability and maintainability
Parts:
- removed PP_EIS_LOAD_A: PP_EIS_LOAD_A, Probe_1.27mm
- removed PP_EIS_LOAD_B: PP_EIS_LOAD_B, Probe_1.27mm
- added R_EIS_LOAD: R_EIS_LOAD, EIS_Load_0603, F.Cu at (72.0, 32.5)

Commit message: Refactor code structure for improved readability and maintainability
Parts:
- moved PP_NTC1 2.30 mm to (15.2, 76.8)
- moved TH1 2.30 mm to (17.7, 76.8)
- moved PP_NTC2 2.30 mm to (35.2, 76.8)
- moved PP_NTC3 2.30 mm to (55.2, 76.8)
- moved PP_NTC4 2.30 mm to (75.2, 76.8)
- moved TH2 2.30 mm to (37.7, 76.8)
- moved TH3 2.30 mm to (57.7, 76.8)
- moved TH4 2.30 mm to (77.7, 76.8)
Routing:
- net NTC3: track 65.7 -> 68.0 mm
- net NTC4: track 66.0 -> 68.3 mm
- net NTC2: track 65.4 -> 67.7 mm
- net NTC1: track 65.5 -> 67.4 mm

Commit message: Refactor code structure for improved readability and maintainability
Parts:
- moved TLM_W0.5 2.00 mm to (48.0, 50.5)
Other:
- board text added: "spacings: 100 / 150 / 250 / 500 / 1000 / 2000 um"
- board text removed: "spacings: 5 / 10 / 20 / 50 / 100 / 200 um"

Commit message: Refactor code structure for improved readability and maintainability
Parts:
- moved PP_EIS_OPEN_A 7.11 mm to (44.5, 35.4)
- moved PP_EIS_OPEN_B 7.11 mm to (47.5, 35.4)
- moved R_EIS_LOAD 4.54 mm to (75.5, 35.4)
- moved PP_EIS_SHORT_A 3.26 mm to (59.5, 35.4)
- moved PP_EIS_SHORT_B 3.26 mm to (62.5, 35.4)
- moved TLM_W0.5 2.00 mm to (50.0, 50.5)
Other:
- board text added: "spacings: 200 / 300 / 500 / 1000 / 2000 / 4000 um"
- board text added: "use: bare-ENIG QC / solder-paste sheet-R after reflow"
- board text removed: "spacings: 100 / 150 / 250 / 500 / 1000 / 2000 um"

Commit message: Refactor code structure for improved readability and maintainability
Parts:
- removed VDP_W0.1: VDP_W0.1, VDP
- added VDP_W0.15: VDP_W0.15, VDP, F.Cu at (83.0, 61.5)
Other:
- board text added: "use: bare-ENIG sheet-R QC (4-probe per cloverleaf, no LED bond)"

Commit message: Refactor code structure for improved readability and maintainability
Other:
- board text added: "bare-ENIG QC | L→R sizes: W=1.0 / 0.5 / 0.25 / 0.15 mm"
- board text removed: "use: bare-ENIG sheet-R QC (4-probe per cloverleaf, no LED bond)"
