File: new-pcb/tud-microled-v2.kicad_pcb (KiCad board)
At the start: 2 copper layers, 93 x 93 mm, 130 parts

Commit message: Finalize PCB for Eurocircuits order: - Updated Yageo resistor MPN from RT0603BRD07100RL to RT0603BRB07100RL for better availability and performance. - Added 3D model references for various footprints in the KiCad PCB file to enhance visualization in the 3D viewer. - Adjusted BOM generation script to reflect the updated resistor MPN. - Compressed project files to include the latest changes.
Parts:
- R_EIS_LOAD: value RT0603BRD07100RL -> RT0603BRB07100RL
Changed lines of the file:
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@@
 		)
 		(embedded_fonts no)
+		(model "${WE_3DMODEL_DIR}/LED_SMD_Wurth.3dshapes/D_Wurth_WL-SFCC-0404superflat.step"
+			(offset (xyz 0 0 0))
+			(scale (xyz 1 1 1))
+			(rotate (xyz 0 0 0))
+		)
 	)
 	(footprint "BondPad_DoE"
@@
 		)
 		(embedded_fonts no)
+		(model "${WE_3DMODEL_DIR}/LED_SMD_Wurth.3dshapes/D_Wurth_WL-SFCC-0404superflat.step"
+			(offset (xyz 0 0 0))
+			(scale (xyz 1 1 1))
+			(rotate (xyz 0 0 0))
+		)
 	)
 	(footprint "Probe_1.27mm"
@@
 		)
 		(embedded_fonts no)
+		(model "${WE_3DMODEL_DIR}/LED_SMD_Wurth.3dshapes/D_Wurth_WL-SFCC-0404superflat.step"
+			(offset (xyz 0 0 0))
+			(scale (xyz 1 1 1))
+			(rotate (xyz 0 0 0))
+		)
 	)
 	(footprint "BondPad_DoE"
@@
 		)
 		(embedded_fonts no)
+		(model "${WE_3DMODEL_DIR}/LED_SMD_Wurth.3dshapes/D_Wurth_WL-SFCC-0404superflat.step"
+			(offset (xyz 0 0 0))
+			(scale (xyz 1 1 1))
+			(rotate (xyz 0 0 0))
+		)
 	)
 	(footprint "Probe_1.27mm"
@@
 		)
 		(embedded_fonts no)
+		(model "${WE_3DMODEL_DIR}/LED_SMD_Wurth.3dshapes/D_Wurth_WL-SFCC-0404superflat.step"
+			(offset (xyz 0 0 0))
+			(scale (xyz 1 1 1))
+			(rotate (xyz 0 0 0))
+		)
 	)
 	(footprint "Probe_1.27mm"
@@
 		)
 		(embedded_fonts no)
+		(model "${WE_3DMODEL_DIR}/LED_SMD_Wurth.3dshapes/D_Wurth_WL-SFCC-0404superflat.step"
+			(offset (xyz 0 0 0))
+			(scale (xyz 1 1 1))
+			(rotate (xyz 0 0 0))
+		)
 	)
 	(footprint "Probe_1.27mm"
@@
 		)
 		(embedded_fonts no)
+		(model "${WE_3DMODEL_DIR}/LED_SMD_Wurth.3dshapes/D_Wurth_WL-SFCC-0404superflat.step"
+			(offset (xyz 0 0 0))
+			(scale (xyz 1 1 1))
+			(rotate (xyz 0 0 0))
+		)
 	)
 	(footprint "WL-SFCC_0404"
@@
 		)
 		(embedded_fonts no)
+		(model "${WE_3DMODEL_DIR}/LED_SMD_Wurth.3dshapes/D_Wurth_WL-SFCC-0404superflat.step"
+			(offset (xyz 0 0 0))
+			(scale (xyz 1 1 1))
+			(rotate (xyz 0 0 0))
+		)
 	)
 	(footprint "Probe_1.27mm"
@@
 		)
 		(embedded_fonts no)
+		(model "${WE_3DMODEL_DIR}/LED_SMD_Wurth.3dshapes/D_Wurth_WL-SFCC-0404superflat.step"
+			(offset (xyz 0 0 0))
+			(scale (xyz 1 1 1))
+			(rotate (xyz 0 0 0))
+		)
 	)
 	(footprint "TLM"
@@
 		)
 		(embedded_fonts no)
+		(model "${KICAD9_3DMODEL_DIR}/Resistor_SMD.3dshapes/R_0402_1005Metric.step"
+			(offset (xyz 0 0 0))
+			(scale (xyz 1 1 1))
+			(rotate (xyz 0 0 0))
+		)
 	)
 	(footprint "Probe_1.27mm"
@@
 		)
 		(embedded_fonts no)
+		(model "${WE_3DMODEL_DIR}/LED_SMD_Wurth.3dshapes/D_Wurth_WL-SFCC-0404superflat.step"
+			(offset (xyz 0 0 0))
+			(scale (xyz 1 1 1))
+			(rotate (xyz 0 0 0))
+		)
 	)
 	(footprint "Probe_1.27mm"
@@
 		)
 		(embedded_fonts no)
+		(model "${WE_3DMODEL_DIR}/LED_SMD_Wurth.3dshapes/D_Wurth_WL-SFCC-0404superflat.step"
+			(offset (xyz 0 0 0))
+			(scale (xyz 1 1 1))
+			(rotate (xyz 0 0 0))
+		)
 	)
 	(footprint "BondPad_DoE"
@@
 		)
 		(embedded_fonts no)
+		(model "${WE_3DMODEL_DIR}/LED_SMD_Wurth.3dshapes/D_Wurth_WL-SFCC-0404superflat.step"
+			(offset (xyz 0 0 0))
+			(scale (xyz 1 1 1))
+			(rotate (xyz 0 0 0))
+		)
 	)
 	(footprint "Probe_1.27mm"
@@
 		)
 		(embedded_fonts no)
+		(model "${WE_3DMODEL_DIR}/LED_SMD_Wurth.3dshapes/D_Wurth_WL-SFCC-0404superflat.step"
+			(offset (xyz 0 0 0))
+			(scale (xyz 1 1 1))
+			(rotate (xyz 0 0 0))
+		)
 	)
 	(footprint "EIS_Load_0603"
@@
 			)
 		)
-		(property "Value" "RT0603BRD07100RL"
+		(property "Value" "RT0603BRB07100RL"
 			(at 0 2 0)
 			(layer "F.Fab")
@@
 			)
 		)
-		(property "MPN" "RT0603BRD07100RL"
+		(property "MPN" "RT0603BRB07100RL"
 			(at 0 0 0)
 			(unlocked yes)
@@
 		)
 		(embedded_fonts no)
+		(model "${KICAD9_3DMODEL_DIR}/Resistor_SMD.3dshapes/R_0603_1608Metric.step"
+			(offset (xyz 0 0 0))
+			(scale (xyz 1 1 1))
+			(rotate (xyz 0 0 0))
+		)
 	)
 	(footprint "WL-SFCC_0404"
@@
 		)
 		(embedded_fonts no)
+		(model "${WE_3DMODEL_DIR}/LED_SMD_Wurth.3dshapes/D_Wurth_WL-SFCC-0404superflat.step"
+			(offset (xyz 0 0 0))
+			(scale (xyz 1 1 1))
+			(rotate (xyz 0 0 0))
+		)
 	)
 	(footprint "Probe_1.27mm"
@@
 		)
 		(embedded_fonts no)
+		(model "${WE_3DMODEL_DIR}/LED_SMD_Wurth.3dshapes/D_Wurth_WL-SFCC-0404superflat.step"
+			(offset (xyz 0 0 0))
+			(scale (xyz 1 1 1))
+			(rotate (xyz 0 0 0))
+		)
 	)
 	(footprint "TLM"
@@
 		)
 		(embedded_fonts no)
+		(model "${WE_3DMODEL_DIR}/LED_SMD_Wurth.3dshapes/D_Wurth_WL-SFCC-0404superflat.step"
+			(offset (xyz 0 0 0))
+			(scale (xyz 1 1 1))
+			(rotate (xyz 0 0 0))
+		)
 	)
 	(footprint "WL-SFCC_0404"
@@
 		)
 		(embedded_fonts no)
+		(model "${WE_3DMODEL_DIR}/LED_SMD_Wurth.3dshapes/D_Wurth_WL-SFCC-0404superflat.step"
+			(offset (xyz 0 0 0))
+			(scale (xyz 1 1 1))
+			(rotate (xyz 0 0 0))
+		)
 	)
 	(footprint "Probe_1.27mm"
@@
 		)
 		(embedded_fonts no)
+		(model "${WE_3DMODEL_DIR}/LED_SMD_Wurth.3dshapes/D_Wurth_WL-SFCC-0404superflat.step"
+			(offset (xyz 0 0 0))
+			(scale (xyz 1 1 1))
+			(rotate (xyz 0 0 0))
+		)
 	)
 	(footprint "TC_Pad_1mm"
@@
 		)
 		(embedded_fonts no)
+		(model "${KICAD9_3DMODEL_DIR}/Resistor_SMD.3dshapes/R_0402_1005Metric.step"
+			(offset (xyz 0 0 0))
+			(scale (xyz 1 1 1))
+			(rotate (xyz 0 0 0))
+		)
 	)
 	(footprint "BondPad_DoE"
@@
 		)
 		(embedded_fonts no)
+		(model "${WE_3DMODEL_DIR}/LED_SMD_Wurth.3dshapes/D_Wurth_WL-SFCC-0404superflat.step"
+			(offset (xyz 0 0 0))
+			(scale (xyz 1 1 1))
+			(rotate (xyz 0 0 0))
+		)
 	)
 	(footprint "BondPad_DoE"
@@
 		)
 		(embedded_fonts no)
+		(model "${KICAD9_3DMODEL_DIR}/Resistor_SMD.3dshapes/R_0402_1005Metric.step"
+			(offset (xyz 0 0 0))
+			(scale (xyz 1 1 1))
+			(rotate (xyz 0 0 0))
+		)
 	)
 	(footprint "Probe_1.27mm"
@@
 		)
 		(embedded_fonts no)
+		(model "${WE_3DMODEL_DIR}/LED_SMD_Wurth.3dshapes/D_Wurth_WL-SFCC-0404superflat.step"
+			(offset (xyz 0 0 0))
+			(scale (xyz 1 1 1))
+			(rotate (xyz 0 0 0))
+		)
 	)
 	(footprint "Fiducial_1mm"
@@
 		)
 		(embedded_fonts no)
+		(model "${WE_3DMODEL_DIR}/LED_SMD_Wurth.3dshapes/D_Wurth_WL-SFCC-0404superflat.step"
+			(offset (xyz 0 0 0))
+			(scale (xyz 1 1 1))
+			(rotate (xyz 0 0 0))
+		)
 	)
 	(footprint "Probe_1.27mm"
@@
 		)
 		(embedded_fonts no)
+		(model "${WE_3DMODEL_DIR}/LED_SMD_Wurth.3dshapes/D_Wurth_WL-SFCC-0404superflat.step"
+			(offset (xyz 0 0 0))
+			(scale (xyz 1 1 1))
+			(rotate (xyz 0 0 0))
+		)
 	)
 	(footprint "Probe_1.27mm"
@@
 		)
 		(embedded_fonts no)
+		(model "${WE_3DMODEL_DIR}/LED_SMD_Wurth.3dshapes/D_Wurth_WL-SFCC-0404superflat.step"
+			(offset (xyz 0 0 0))
+			(scale (xyz 1 1 1))
+			(rotate (xyz 0 0 0))
+		)
 	)
 	(footprint "Probe_1.27mm"
@@
 		)
 		(embedded_fonts no)
+		(model "${WE_3DMODEL_DIR}/LED_SMD_Wurth.3dshapes/D_Wurth_WL-SFCC-0404superflat.step"
+			(offset (xyz 0 0 0))
+			(scale (xyz 1 1 1))
+			(rotate (xyz 0 0 0))
+		)
 	)
 	(footprint "Probe_1.27mm"
@@
 		)
 		(embedded_fonts no)
+		(model "${WE_3DMODEL_DIR}/LED_SMD_Wurth.3dshapes/D_Wurth_WL-SFCC-0404superflat.step"
+			(offset (xyz 0 0 0))
+			(scale (xyz 1 1 1))
+			(rotate (xyz 0 0 0))
+		)
 	)
 	(footprint "Probe_1.27mm"
@@
 		)
 		(embedded_fonts no)
+		(model "${WE_3DMODEL_DIR}/LED_SMD_Wurth.3dshapes/D_Wurth_WL-SFCC-0404superflat.step"
+			(offset (xyz 0 0 0))
+			(scale (xyz 1 1 1))
+			(rotate (xyz 0 0 0))
+		)
 	)
 	(footprint "BondPad_DoE"
@@
 		)
 		(embedded_fonts no)
+		(model "${KICAD9_3DMODEL_DIR}/Resistor_SMD.3dshapes/R_0402_1005Metric.step"
+			(offset (xyz 0 0 0))
+			(scale (xyz 1 1 1))
+			(rotate (xyz 0 0 0))
+		)
 	)
 	(footprint "Probe_1.27mm"
@@
 		)
 		(embedded_fonts no)
+		(model "${KICAD9_3DMODEL_DIR}/Connector_PinHeader_2.54mm.3dshapes/PinHeader_1x32_P2.54mm_Vertical.step"
+			(offset (xyz 0 0 0))
+			(scale (xyz 1 1 1))
+			(rotate (xyz 0 0 -90))
+		)
 	)
 	(footprint "Header_2.54mm"
@@
 		)
 		(embedded_fonts no)
+		(model "${KICAD9_3DMODEL_DIR}/Connector_PinHeader_2.54mm.3dshapes/PinHeader_1x32_P2.54mm_Vertical.step"
+			(offset (xyz 0 0 0))
+			(scale (xyz 1 1 1))
+			(rotate (xyz 0 0 -90))
+		)
 	)
 	(gr_line
