File: new-pcb/tud-microled-v2.kicad_sch (KiCad schematic)
At the start: 0 parts

Commit message: Refactor code structure for improved readability and maintainability
Parts:
- added D1, D2, D3, D4, D5, D6, D7, D8, DCL12_L1, DCL12_L10, DCL12_L11, DCL12_L12, DCL12_L2, DCL12_L3, DCL12_L4, DCL12_L5, DCL12_L6, DCL12_L7, DCL12_L8, DCL12_L9, DCL6_L1, DCL6_L2, DCL6_L3, DCL6_L4, DCL6_L5, DCL6_L6: WL-SFCC RGB, LED_SMD_Wurth:D_Wurth_WL-SFCC-0404superflat, symbol Device:LED
- added J_N: H_N 1x32 hdr (chain+NTC+jumpers), TUD-microLED:Header_2.54mm, symbol Connector_Generic:Conn_01x32
- added J_S: H_S 1x32 hdr (LED outputs), TUD-microLED:Header_2.54mm, symbol Connector_Generic:Conn_01x32
- added R_EIS_LOAD: 100R 0.1% TNPW0603100RBEEA, TUD-microLED:EIS_Load_0603, symbol Device:R
- added TH1, TH2, TH3, TH4: 10k NCP15XH103J03RC, TUD-microLED:NTC_0402, symbol Device:Thermistor_NTC
- added TP_EIS_OPEN_A: EIS OPEN A, TUD-microLED:Probe_1.27mm, symbol Connector:TestPoint
- added TP_EIS_OPEN_B: EIS OPEN B, TUD-microLED:Probe_1.27mm, symbol Connector:TestPoint
- added TP_EIS_SHORT: EIS SHORT, TUD-microLED:Probe_1.27mm, symbol Connector:TestPoint
Connections:
- new net DCL12_IN: DCL12_L1.2 (A), J_N.19 (Pin_19)
- new net DCL12_J1: DCL12_L1.1 (K), DCL12_L2.2 (A)
- new net DCL12_J10: DCL12_L10.1 (K), DCL12_L11.2 (A)
- new net DCL12_J11: DCL12_L11.1 (K), DCL12_L12.2 (A)
- new net DCL12_J2: DCL12_L2.1 (K), DCL12_L3.2 (A)
- new net DCL12_J3: DCL12_L3.1 (K), DCL12_L4.2 (A)
- new net DCL12_J4: DCL12_L4.1 (K), DCL12_L5.2 (A)
- new net DCL12_J5: DCL12_L5.1 (K), DCL12_L6.2 (A)
- new net DCL12_J6: DCL12_L6.1 (K), DCL12_L7.2 (A)
- new net DCL12_J7: DCL12_L7.1 (K), DCL12_L8.2 (A)
- new net DCL12_J8: DCL12_L8.1 (K), DCL12_L9.2 (A)
- new net DCL12_J9: DCL12_L10.2 (A), DCL12_L9.1 (K)
- new net DCL12_OUT: DCL12_L12.1 (K), J_N.32 (Pin_32)
- new net DCL6_IN: DCL6_L1.2 (A), J_N.3 (Pin_3)
- new net DCL6_J1: DCL6_L1.1 (K), DCL6_L2.2 (A)
- new net DCL6_J2: DCL6_L2.1 (K), DCL6_L3.2 (A)
- new net DCL6_J3: DCL6_L3.1 (K), DCL6_L4.2 (A)
- new net DCL6_J4: DCL6_L4.1 (K), DCL6_L5.2 (A)
- new net DCL6_J5: DCL6_L5.1 (K), DCL6_L6.2 (A)
- new net DCL6_OUT: DCL6_L6.1 (K), J_N.10 (Pin_10)
- new net EIS_LOAD_A: R_EIS_LOAD.1
- new net EIS_LOAD_B: R_EIS_LOAD.2
- new net EIS_OPEN_A: TP_EIS_OPEN_A.1
- new net EIS_OPEN_B: TP_EIS_OPEN_B.1
- new net EIS_SHORT: TP_EIS_SHORT.1
- new net GND: TH1.2, TH2.2, TH3.2, TH4.2
- new net LED1_KB: J_S.3 (Pin_3)
- new net LED1_KG: J_S.2 (Pin_2)
- new net LED1_KR: D1.1 (K), J_S.4 (Pin_4)
- new net LED2_KB: J_S.7 (Pin_7)
- new net LED2_KG: J_S.6 (Pin_6)
- new net LED2_KR: D2.1 (K), J_S.8 (Pin_8)
- new net LED3_KB: J_S.11 (Pin_11)
- new net LED3_KG: J_S.10 (Pin_10)
- new net LED3_KR: D3.1 (K), J_S.12 (Pin_12)
- new net LED4_KB: J_S.15 (Pin_15)
- new net LED4_KG: J_S.14 (Pin_14)
- new net LED4_KR: D4.1 (K), J_S.16 (Pin_16)
- new net LED5_KB: J_S.19 (Pin_19)
- new net LED5_KG: J_S.18 (Pin_18)
- new net LED5_KR: D5.1 (K), J_S.20 (Pin_20)
- new net LED6_KB: J_S.23 (Pin_23)
- new net LED6_KG: J_S.22 (Pin_22)
- new net LED6_KR: D6.1 (K), J_S.24 (Pin_24)
- new net LED7_KB: J_S.27 (Pin_27)
- new net LED7_KG: J_S.26 (Pin_26)
- new net LED7_KR: D7.1 (K), J_S.28 (Pin_28)
- new net LED8_KB: J_S.31 (Pin_31)
- new net LED8_KG: J_S.30 (Pin_30)
- new net LED8_KR: D8.1 (K), J_S.32 (Pin_32)
- new net LED_VCC: D1.2 (A), D2.2 (A), D3.2 (A), D4.2 (A), D5.2 (A), D6.2 (A), D7.2 (A), D8.2 (A), J_S.1 (Pin_1), J_S.13 (Pin_13), J_S.17 (Pin_17), J_S.21 (Pin_21), J_S.25 (Pin_25), J_S.29 (Pin_29), J_S.5 (Pin_5), J_S.9 (Pin_9)
- new net NTC1: J_N.5 (Pin_5), TH1.1
- new net NTC2: J_N.13 (Pin_13), TH2.1
- new net NTC3: J_N.21 (Pin_21), TH3.1
- new net NTC4: J_N.29 (Pin_29), TH4.1
- no-connect marks 0 -> 24
Other:
- note added: "BLOCK 1 — LED MATRIX D1–D8 (8 × Wurth WL-SFCC RGB common-anode) → cathodes route to south header H_S_1..32"
- note added: "BLOCK 2 — DCL6 DAISY CHAIN (6 × WL-SFCC, A→K_R series) · K_G / K_B per LED isolated (probe-only) · endpoints route to H_N_3 / H_N_10"
- note added: "BLOCK 3 — DCL12 DAISY CHAIN (12 × WL-SFCC, A→K_R series) · endpoints route to H_N_19 / H_N_32"
- note added: "BLOCK 4 — NTC THERMISTORS (TH1–TH4, Murata NCP15XH103J03RC, 10 kΩ ±5 %, B25/85 = 3380 K) → V_F-TSP thermal sensing of bonded LEDs"
- note added: "BLOCK 5 — EIS CALIBRATION (LCR-meter Nyquist reference: 100 Ω LOAD + OPEN (∞) + SHORT (0 Ω))"
- note added: "BLOCK 6 — HEADERS (2 × Wurth WR-PHD 61304011121, 1×32 single-row male, 2.54 mm pitch, vertical THT)"
- note added: "DESIGN NOTES — Test structures (bare ENIG pads, no electrical connections, not shown on schematic):"
- note added: "NET NAMING: LED_VCC = common anode bus · LEDn_K{R,G,B} = cathode of D1..D8 · DCL{6,12}_IN/OUT = chain endpoints · DCL{6,12}_Jk = chain junction k · DCLn_Lk_K{G,B} = isolated G/B cathodes (chain LEDs, probe-only) · NTCn = thermistor sense · EIS_LOAD_A/B = 100 Ω cal resistor · EIS_OPEN_A/B = open-circuit cal · EIS_SHORT = short-circuit cal · GND = common return"
- note added: "PCB-side notes: WL-SFCC LEDs depicted with single Device:LED symbol per chip — K shown = K_R (in-chain cathode); K_G and K_B route to PCB pads via labels and reach the south header at pins (4k+2) and (4k+3)."
- note added: "• DoE bond-pad array (36 × isolated 1 mm pads, 3.5 mm pitch) • TLM ladders (3 widths × 7 fingers, 200/300/500/1000/2000/4000 µm gaps)"
- note added: "• Thermocouple pads TC1-4 (in-situ reflow temp) • Optical fiducials FID1-4 (P&P alignment)"
- note added: "• Van der Pauw cloverleaves (W=1.0/0.5/0.25/0.15 mm × 4 contacts) • Probe pads PP_* (46): 4-wire access to bonded LEDs"
- company: (none) -> TU Delft · ECTM + ITEC
- title: (none) -> TUD Micro-LED Bond Characterization — v4.0.7 PCB
Changed lines of the file:
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@@
-(kicad_sch (version 20250114) (generator "KiCAD-MCP-Server")
-  (paper "A4")
-  (sheet_instances
-    (path "/" (page "1"))
-  )
-)
